File: RPiPicoKlipperAsciiHMI/RPiPicoKlipperAsciiHMI.kicad_sch (KiCad schematic)
At the start: 14 parts, among them SW1 KILL, SW2 BACK, SW3 UP, SW4 DOWN, U1 LCD-20X4, U2 Pico, U3 ROTARY_ENCODER_MODULE, U4 ULN2803A

Commit message: Added latest Version of POC KiCAD Project
Parts:
- added R? (x8): 200, symbol Device:R
Connections:
- net +3V3: now also U2.36 (3V3)
- net GND: now also U2.38 (GND); no longer U2.39 (VSYS)
- new net ButtonBoard/BTN1_LED+: R?.1
- new net ButtonBoard/BTN2_LED+: R?.2
- new net ButtonBoard/BTN3_LED+: R?.1
- new net ButtonBoard/BTN4_LED+: R?.2
- new net ButtonBoard/BTN5_LED+: R?.2
- new net ButtonBoard/BTN6_LED+: R?.2
- new net ButtonBoard/BTN7_LED+: R?.1
- new net ButtonBoard/BTN8_LED+: R?.1
Other:
- added sheet ButtonBoard (ButtonBoard.kicad_sch)
- note added: "Optional Can be connected directly to GND if no controlling of LCD BG-LED Brightness is needed"
- note removed: "Optional Can be connected directly to GND if now controlling of LCD BG-LED Brightness is needed"
